Commit message: Update radius value

File: two_wheeled/src/m2wr_description/urdf/m2wr.xacro (robot description, xacro)
@@ -90,5 +90,5 @@
       <origin rpy="0 1.5707 1.5707" xyz="0 0 0" />
       <geometry>
-        <cylinder length="0.04" radius="0.1"/>
+        <cylinder length="0.04" radius="0.5"/>
       </geometry>
     </collision>
@@ -96,5 +96,5 @@
       <origin rpy="0 1.5707 1.5707" xyz="0 0 0"/>
       <geometry>
-        <cylinder length="0.04" radius="0.1"/>
+        <cylinder length="0.04" radius="0.5"/>
       </geometry>
     </visual>
@@ -123,5 +123,5 @@
       <origin rpy="0 1.5707 1.5707" xyz="0 0 0" />
       <geometry>
-        <cylinder length="0.04" radius="0.1"/>
+        <cylinder length="0.04" radius="0.5"/>
       </geometry>
     </collision>
@@ -129,5 +129,5 @@
       <origin rpy="0 1.5707 1.5707" xyz="0 0 0"/>
       <geometry>
-        <cylinder length="0.04" radius="0.1"/>
+        <cylinder length="0.04" radius="0.5"/>
       </geometry>
     </visual>
